File: pcb/fw-anwesenheit.kicad_sch (KiCad schematic)
At the start: 47 parts, among them J1 Conn_01x02_Pin, J2 I2C, J3 LED, J4 MicroSD, U1 XIAO-ESP32-S3-SMD, U2 SN74AHCT1G125DBVT, U4 DS3232M

Commit message: pcb v1 finish
Parts:
- removed J3: LED, Connector_PinHeader_2.54mm:PinHeader_1x04_P2.54mm_Vertical, symbol Connector:Conn_01x04_Pin
- added J3: LED, Connector_PinSocket_2.00mm:PinSocket_1x03_P2.00mm_Vertical, symbol Connector:Conn_01x03_Pin
- BZ1: footprint Connector_PinHeader_2.54mm:PinHeader_1x02_P2.54mm_Vertical -> Connector_PinSocket_2.00mm:PinSocket_1x02_P2.00mm_Vertical
- D2: footprint (none) -> LED_SMD:LED_0603_1608Metric
- JP1: value Li-IOn Enable -> Li-Ion
- R7, R8: now not fitted
- TP14: value 3,3V -> DAT1
- TP15: value 3,3V -> DAT2
- TP5: value Din -> CS
- TP6: value Dout -> SD_DECT
Connections:
- net +3.3V: now also D2.2 (A); no longer R1.2
- net +5V: now also J3.2 (Pin_2)
- net GND: now also J3.3 (Pin_3)
- net LED_Din: now also J3.1 (Pin_1); no longer TP5.1
- net SD_DECT: now also TP6.1
- net SPI_CS: now also TP5.1
- net at BT1.1 (+), U4.6 (VBAT): no longer J1.1 (Pin_1), JP1.2 (B)
- net at D2.1 (K): now also R1.2; no longer RDM1.LED
- net at R1.1: now also RDM1.LED; no longer D2.2 (A)
- new net: J1.1 (Pin_1), JP1.2 (B)
Other:
- moved on the sheet: D2, R1
