File: pcb/fw-anwesenheit.kicad_sch (KiCad schematic)
At the start: 48 parts, among them J1 Conn_01x02_Pin, J2 I2C, J3 LED, J4 MicroSD, U1 XIAO-ESP32-S3-SMD, U2 SN74AHCT1G125DBVT, U3 DS3231M

Commit message: changed some pcb descriptions and Resistor for LED
Parts:
- C2, C3: value 100 nF -> 100nF
- R1: value 100R -> 150R
Changed lines of the file:
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@@
 			)
 		)
-		(property "Value" "100 nF"
+		(property "Value" "100nF"
 			(at 105.41 166.3699 0)
 			(effects
@@
 			)
 		)
-		(property "Value" "100 nF"
+		(property "Value" "100nF"
 			(at 200.66 135.8899 0)
 			(effects
@@
 			)
 		)
-		(property "Value" "100R"
+		(property "Value" "150R"
 			(at 140.97 91.44 90)
 			(effects

Commit message: fixed buzzer footprint
Parts:
- BZ1: footprint Connector_PinSocket_2.00mm:PinSocket_1x02_P2.00mm_Vertical -> Connector_PinSocket_2.54mm:PinSocket_1x02_P2.54mm_Vertical
Changed lines of the file:
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@@
 			)
 		)
-		(property "Footprint" "Connector_PinSocket_2.00mm:PinSocket_1x02_P2.00mm_Vertical"
+		(property "Footprint" "Connector_PinSocket_2.54mm:PinSocket_1x02_P2.54mm_Vertical"
 			(at 203.835 21.59 90)
 			(effects
