File: pcb/fw-anwesenheit-backups/fw-anwesenheit-2025-08-22_211436/fw-anwesenheit.kicad_pcb (KiCad board)
At the start: 6 copper layers, 50 x 50 mm, 48 parts, among them J1 Conn_01x02_Pin, J2 I2C, J3 LED, J4 MicroSD, U1 XIAO-ESP32-S3-SMD, U2 SN74AHCT1G125DBVT, U3 DS3231M

Commit message: fixed RTC footprint and some labels
Parts:
- R1, R2: value 100R -> 100
- moved BT1 0.89 mm to (112.5, 103.4)
- moved J3 0.23 mm to (129.0, 111.2)
- moved R5 0.07 mm to (120.0, 120.1)
Routing:
- net +3.3V: track 27.7 -> 4.05 mm, vias 41 -> 31
- net GND: vias 107 -> 102
Other:
- board text added: "3,3V GND SDA SCL"
- board text removed: "3.3V GND SDA SCL"
- board text removed: "Buzzer"
- board text removed: "Designed for external Antenna"
